File: kicad/Extension.kicad_sch (KiCad schematic)
At the start: 2 parts, among them J3 FTS-126-02-L-DV, U1 LFE5U-25F-6BG381C

Commit message: Update Extension.kicad_sch
Other:
- note added: "Extension Connector"
Changed lines of the file:
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@@
 		)
 	)
-	(text "Extension"
+	(text "Extension Connector"
 		(exclude_from_sim no)
 		(at 178.308 172.72 0)

Commit message: Routing complete
Other:
- moved on the sheet: J3, U1B, U1C, U1G

Commit message: Changed the name of the project path
Parts:
- J3: footprint ECP5_TX_AUDIO:SAMTEC-FTS-126-02-X-DV -> ECP5_BGA381_FT2232HQ_FIFO:SAMTEC-FTS-126-02-X-DV
- U1: footprint ECP5_TX_AUDIO:BGA-381_pitch0.8mm_dia0.4mm -> ECP5_BGA381_FT2232HQ_FIFO:BGA-381_pitch0.8mm_dia0.4mm; symbol ECP5_TX_AUDIO:LFE5U-25F-xBG381x -> ECP5_BGA381_FT2232HQ_FIFO:LFE5U-25F-xBG381x
Changed lines of the file:
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@@
 	)
 	(symbol
-		(lib_id "ECP5_TX_AUDIO:LFE5U-25F-xBG381x")
+		(lib_id "ECP5_BGA381_FT2232HQ_FIFO:LFE5U-25F-xBG381x")
 		(at 179.07 59.69 0)
 		(unit 2)
@@
 			)
 		)
-		(property "Footprint" "ECP5_TX_AUDIO:BGA-381_pitch0.8mm_dia0.4mm"
+		(property "Footprint" "ECP5_BGA381_FT2232HQ_FIFO:BGA-381_pitch0.8mm_dia0.4mm"
 			(at 175.26 -97.79 0)
 			(effects
@@
 	)
 	(symbol
-		(lib_id "ECP5_TX_AUDIO:LFE5U-25F-xBG381x")
+		(lib_id "ECP5_BGA381_FT2232HQ_FIFO:LFE5U-25F-xBG381x")
 		(at 147.32 59.69 0)
 		(unit 7)
@@
 			)
 		)
-		(property "Footprint" "ECP5_TX_AUDIO:BGA-381_pitch0.8mm_dia0.4mm"
+		(property "Footprint" "ECP5_BGA381_FT2232HQ_FIFO:BGA-381_pitch0.8mm_dia0.4mm"
 			(at 143.51 -97.79 0)
 			(effects
@@
 			)
 		)
-		(property "Footprint" "ECP5_TX_AUDIO:SAMTEC-FTS-126-02-X-DV"
+		(property "Footprint" "ECP5_BGA381_FT2232HQ_FIFO:SAMTEC-FTS-126-02-X-DV"
 			(at 59.69 66.04 0)
 			(effects
@@
 	)
 	(symbol
-		(lib_id "ECP5_TX_AUDIO:LFE5U-25F-xBG381x")
+		(lib_id "ECP5_BGA381_FT2232HQ_FIFO:LFE5U-25F-xBG381x")
 		(at 111.76 63.5 0)
 		(unit 3)
@@
 			)
 		)
-		(property "Footprint" "ECP5_TX_AUDIO:BGA-381_pitch0.8mm_dia0.4mm"
+		(property "Footprint" "ECP5_BGA381_FT2232HQ_FIFO:BGA-381_pitch0.8mm_dia0.4mm"
 			(at 107.95 -93.98 0)
 			(effects
