File: kicad/FT2232HQ_FIFO.kicad_sch (KiCad schematic)
At the start: 41 parts, among them J2 USB Type C, U1 LFE5U-25F-6BG381C, U4 LP5907MFX-3.3, U5 FT2232HQ, U6 93LCxxBxxOT, Y2 12.000 MHz

Commit message: Updated the names of the Sheets
Other:
- note added: "FT2232HQ FIFO Interface"
- note removed: "FT2232HQ & Extension Connector"
Changed lines of the file:
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@@
 		)
 	)
-	(text "FT2232HQ & Extension Connector"
+	(text "FT2232HQ FIFO Interface"
 		(exclude_from_sim no)
 		(at 178.816 172.466 0)

Commit message: Routing complete
Parts:
- renumbered C10 to C11, C11 to C12, C12 to C13, C13 to C14, C14 to C15, C15 to C16, C16 to C17, C17 to C18, C18 to C19, C19 to C20, C20 to C21, C21 to C22, C22 to C23, C23 to C24, C24 to C25, C25 to C26, C26 to C27, C27 to C28, C28 to C29, C29 to C30, Y2 to Y3

Commit message: PCB changes
Connections:
- net FT2232_RESET renamed ~{FT2232_RESET}
Changed lines of the file:
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@@
 		)
 	)
-	(global_label "FT2232_RESET"
+	(global_label "~{FT2232_RESET}"
 		(shape input)
 		(at 95.25 123.19 180)
@@
 		)
 	)
-	(global_label "FT2232_RESET"
+	(global_label "~{FT2232_RESET}"
 		(shape output)
 		(at 226.06 36.83 180)

Commit message: Changed the name of the project path
Parts:
- F2: footprint ECP5_TX_AUDIO:Fuse_1812_4532Metric -> ECP5_BGA381_FT2232HQ_FIFO:Fuse_1812_4532Metric
- J2: footprint ECP5_TX_AUDIO:USB_C_Receptacle_GCT_USB4105-xx-A_16P_TopMnt_Horizontal -> ECP5_BGA381_FT2232HQ_FIFO:USB_C_Receptacle_GCT_USB4105-xx-A_16P_TopMnt_Horizontal; symbol ECP5_TX_AUDIO:USB_C_Receptacle_USB2.0 -> ECP5_BGA381_FT2232HQ_FIFO:USB_C_Receptacle_USB2.0
- U1: footprint ECP5_TX_AUDIO:BGA-381_pitch0.8mm_dia0.4mm -> ECP5_BGA381_FT2232HQ_FIFO:BGA-381_pitch0.8mm_dia0.4mm; symbol ECP5_TX_AUDIO:LFE5U-25F-xBG381x -> ECP5_BGA381_FT2232HQ_FIFO:LFE5U-25F-xBG381x
Changed lines of the file:
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@@
 	)
 	(symbol
-		(lib_id "ECP5_TX_AUDIO:LFE5U-25F-xBG381x")
+		(lib_id "ECP5_BGA381_FT2232HQ_FIFO:LFE5U-25F-xBG381x")
 		(at 269.24 60.96 0)
 		(unit 4)
@@
 			)
 		)
-		(property "Footprint" "ECP5_TX_AUDIO:BGA-381_pitch0.8mm_dia0.4mm"
+		(property "Footprint" "ECP5_BGA381_FT2232HQ_FIFO:BGA-381_pitch0.8mm_dia0.4mm"
 			(at 265.43 -96.52 0)
 			(effects
@@
 	)
 	(symbol
-		(lib_id "ECP5_TX_AUDIO:USB_C_Receptacle_USB2.0")
+		(lib_id "ECP5_BGA381_FT2232HQ_FIFO:USB_C_Receptacle_USB2.0")
 		(at 24.13 50.8 0)
 		(unit 1)
@@
 			)
 		)
-		(property "Footprint" "ECP5_TX_AUDIO:USB_C_Receptacle_GCT_USB4105-xx-A_16P_TopMnt_Horizontal"
+		(property "Footprint" "ECP5_BGA381_FT2232HQ_FIFO:USB_C_Receptacle_GCT_USB4105-xx-A_16P_TopMnt_Horizontal"
 			(at 27.94 50.8 0)
 			(effects
@@
 			)
 		)
-		(property "Description" "CONN RCP USB2.0 TYP C 24P SMD RA"
+		(property "Description" "USB 2.0-only Type-C Receptacle connector"
 			(at 24.13 50.8 0)
 			(effects
@@
 	)
 	(symbol
-		(lib_id "ECP5_TX_AUDIO:LFE5U-25F-xBG381x")
+		(lib_id "ECP5_BGA381_FT2232HQ_FIFO:LFE5U-25F-xBG381x")
 		(at 237.49 62.23 0)
 		(unit 5)
@@
 			)
 		)
-		(property "Footprint" "ECP5_TX_AUDIO:BGA-381_pitch0.8mm_dia0.4mm"
+		(property "Footprint" "ECP5_BGA381_FT2232HQ_FIFO:BGA-381_pitch0.8mm_dia0.4mm"
 			(at 233.68 -95.25 0)
 			(effects
@@
 			)
 		)
-		(property "Footprint" "ECP5_TX_AUDIO:Fuse_1812_4532Metric"
+		(property "Footprint" "ECP5_BGA381_FT2232HQ_FIFO:Fuse_1812_4532Metric"
 			(at 39.37 36.83 0)
 			(effects
