File: kicad/Flash_JTAG.kicad_sch (KiCad schematic)
At the start: 56 parts, among them J1 USB Type C, Q1 MMST2222A, SW1 User, U1 LFE5U-25F-6BG381C, U2 IS25LP128F, U3 FT231XQ, Y1 50MHz

Commit message: Routing complete
Parts:
- added C2: 0.1µF, Capacitor_SMD:C_0603_1608Metric, symbol Device:C_Small
- added Y2: 22.5792 MHz, Oscillator:Oscillator_SMD_Abracon_ASE-4Pin_3.2x2.5mm, symbol Device:Crystal_GND24
- Y1: value 50MHz -> 24.576 MHz; footprint ECP5_TX_AUDIO:Oscillator_SMD_Diodes_FN-4Pin_7.0x5.0mm -> Oscillator:Oscillator_SMD_Abracon_ASE-4Pin_3.2x2.5mm; MPN ECS-7050MV-500-DM-TR -> 830207659209; Manufacturer ECS Inc. -> Wurth Elektronik
- renumbered C9 to C10, C2 to C3, C3 to C4, C4 to C5, C5 to C6, C6 to C7, C7 to C8, C8 to C9, D7 to D5, D5 to D6, D6 to D7, R20 to R19, R21 to R20, R19 to R21
Connections:
- net +3V3: now also C2.1, Y2.1, Y2.4
- net GND: now also C2.2, Y2.2
- net LED_2: now also U1.F1 (PL26B); no longer U1.H2 (PL26C)
- net CLK_50MHz renamed CLK_24.576MHz
- new net CLK_22.5792MHz: U1.H2 (PL26C), Y2.3
- no-connect marks 28 -> 27
Other:
- moved on the sheet: C1, D3, D4, D6, D7, R14, R15, R16, R17, R21, SW1, U1F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

Commit message: Changed the name of the project path
Parts:
- F1: footprint ECP5_TX_AUDIO:Fuse_1812_4532Metric -> ECP5_BGA381_FT2232HQ_FIFO:Fuse_1812_4532Metric
- J1: footprint ECP5_TX_AUDIO:USB_C_Receptacle_GCT_USB4105-xx-A_16P_TopMnt_Horizontal -> ECP5_BGA381_FT2232HQ_FIFO:USB_C_Receptacle_GCT_USB4105-xx-A_16P_TopMnt_Horizontal; symbol ECP5_TX_AUDIO:USB_C_Receptacle_USB2.0 -> ECP5_BGA381_FT2232HQ_FIFO:USB_C_Receptacle_USB2.0
- U1: footprint ECP5_TX_AUDIO:BGA-381_pitch0.8mm_dia0.4mm -> ECP5_BGA381_FT2232HQ_FIFO:BGA-381_pitch0.8mm_dia0.4mm; symbol ECP5_TX_AUDIO:LFE5U-25F-xBG381x -> ECP5_BGA381_FT2232HQ_FIFO:LFE5U-25F-xBG381x
- U2: footprint ECP5_TX_AUDIO:WSON-8-1EP_6x5mm_P1.27mm_EP3.4x4.3mm -> ECP5_BGA381_FT2232HQ_FIFO:WSON-8-1EP_6x5mm_P1.27mm_EP3.4x4.3mm; symbol ECP5_TX_AUDIO:25LCxxx -> ECP5_BGA381_FT2232HQ_FIFO:25LCxxx
- U3: symbol ECP5_TX_AUDIO:FT231XQ -> ECP5_BGA381_FT2232HQ_FIFO:FT231XQ
Changed lines of the file:
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@@
 	)
 	(symbol
-		(lib_id "ECP5_TX_AUDIO:FT231XQ")
+		(lib_id "ECP5_BGA381_FT2232HQ_FIFO:FT231XQ")
 		(at 101.6 148.59 0)
 		(unit 1)
@@
 			)
 		)
-		(property "Description" "IC USB SERIAL FULL UART 20QFN"
+		(property "Description" "Full Speed USB to Full Handshake UART, QFN-20"
 			(at 101.6 148.59 0)
 			(effects
@@
 	)
 	(symbol
-		(lib_id "ECP5_TX_AUDIO:USB_C_Receptacle_USB2.0")
+		(lib_id "ECP5_BGA381_FT2232HQ_FIFO:USB_C_Receptacle_USB2.0")
 		(at 31.75 140.97 0)
 		(unit 1)
@@
 			)
 		)
-		(property "Footprint" "ECP5_TX_AUDIO:USB_C_Receptacle_GCT_USB4105-xx-A_16P_TopMnt_Horizontal"
+		(property "Footprint" "ECP5_BGA381_FT2232HQ_FIFO:USB_C_Receptacle_GCT_USB4105-xx-A_16P_TopMnt_Horizontal"
 			(at 35.56 140.97 0)
 			(effects
@@
 			)
 		)
-		(property "Description" "CONN RCP USB2.0 TYP C 24P SMD RA"
+		(property "Description" "USB 2.0-only Type-C Receptacle connector"
 			(at 31.75 140.97 0)
 			(effects
@@
 	)
 	(symbol
-		(lib_id "ECP5_TX_AUDIO:LFE5U-25F-xBG381x")
+		(lib_id "ECP5_BGA381_FT2232HQ_FIFO:LFE5U-25F-xBG381x")
 		(at 135.89 45.72 0)
 		(unit 8)
@@
 			)
 		)
-		(property "Footprint" "ECP5_TX_AUDIO:BGA-381_pitch0.8mm_dia0.4mm"
+		(property "Footprint" "ECP5_BGA381_FT2232HQ_FIFO:BGA-381_pitch0.8mm_dia0.4mm"
 			(at 132.08 -111.76 0)
 			(effects
@@
 	)
 	(symbol
-		(lib_id "ECP5_TX_AUDIO:25LCxxx")
+		(lib_id "ECP5_BGA381_FT2232HQ_FIFO:25LCxxx")
 		(at 41.91 71.12 0)
 		(unit 1)
@@
 			)
 		)
-		(property "Footprint" "ECP5_TX_AUDIO:WSON-8-1EP_6x5mm_P1.27mm_EP3.4x4.3mm"
+		(property "Footprint" "ECP5_BGA381_FT2232HQ_FIFO:WSON-8-1EP_6x5mm_P1.27mm_EP3.4x4.3mm"
 			(at 41.91 71.12 0)
 			(effects
@@
 	)
 	(symbol
-		(lib_id "ECP5_TX_AUDIO:LFE5U-25F-xBG381x")
+		(lib_id "ECP5_BGA381_FT2232HQ_FIFO:LFE5U-25F-xBG381x")
 		(at 276.86 69.85 0)
 		(unit 6)
@@
 			)
 		)
-		(property "Footprint" "ECP5_TX_AUDIO:BGA-381_pitch0.8mm_dia0.4mm"
+		(property "Footprint" "ECP5_BGA381_FT2232HQ_FIFO:BGA-381_pitch0.8mm_dia0.4mm"
 			(at 273.05 -87.63 0)
 			(effects
@@
 			)
 		)
-		(property "Footprint" "ECP5_TX_AUDIO:Fuse_1812_4532Metric"
+		(property "Footprint" "ECP5_BGA381_FT2232HQ_FIFO:Fuse_1812_4532Metric"
 			(at 45.72 105.41 0)
 			(effects
@@
 	)
 	(symbol
-		(lib_id "ECP5_TX_AUDIO:LFE5U-25F-xBG381x")
+		(lib_id "ECP5_BGA381_FT2232HQ_FIFO:LFE5U-25F-xBG381x")
 		(at 175.26 121.92 0)
 		(mirror y)
@@
 			)
 		)
-		(property "Footprint" "ECP5_TX_AUDIO:BGA-381_pitch0.8mm_dia0.4mm"
+		(property "Footprint" "ECP5_BGA381_FT2232HQ_FIFO:BGA-381_pitch0.8mm_dia0.4mm"
 			(at 179.07 -35.56 0)
 			(effects
