File: kicad/Power.kicad_sch (KiCad schematic)
At the start: 42 parts, among them U1 LFE5U-25F-6BG381C, U7 TLV62569DBVT, U8 TLV62569DBVT, U9 TLV62569DBVT

Commit message: Routing complete
Parts:
- renumbered C30 to C31, C31 to C32, C32 to C33, C33 to C34, C34 to C35, C35 to C36, C36 to C37, C37 to C38, C38 to C39, C39 to C40, C40 to C41, C41 to C42, C42 to C43, C43 to C44, C44 to C45, C45 to C46, C46 to C47, C47 to C48, C48 to C49, C49 to C50, C50 to C51, C51 to C52, C52 to C53, C53 to C54, C54 to C55, C55 to C56, C56 to C57

Commit message: Changed the name of the project path
Parts:
- TP1, TP2: footprint ECP5_TX_AUDIO:KEYSTONE_5197TR -> ECP5_BGA381_FT2232HQ_FIFO:KEYSTONE_5197TR
- U1: footprint ECP5_TX_AUDIO:BGA-381_pitch0.8mm_dia0.4mm -> ECP5_BGA381_FT2232HQ_FIFO:BGA-381_pitch0.8mm_dia0.4mm; symbol ECP5_TX_AUDIO:LFE5U-25F-xBG381x -> ECP5_BGA381_FT2232HQ_FIFO:LFE5U-25F-xBG381x
Changed lines of the file:
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@@
 			)
 		)
-		(property "Footprint" "ECP5_TX_AUDIO:KEYSTONE_5197TR"
+		(property "Footprint" "ECP5_BGA381_FT2232HQ_FIFO:KEYSTONE_5197TR"
 			(at 34.29 67.31 0)
 			(effects
@@
 			)
 		)
-		(property "Footprint" "ECP5_TX_AUDIO:KEYSTONE_5197TR"
+		(property "Footprint" "ECP5_BGA381_FT2232HQ_FIFO:KEYSTONE_5197TR"
 			(at 24.13 67.31 0)
 			(effects
@@
 	)
 	(symbol
-		(lib_id "ECP5_TX_AUDIO:LFE5U-25F-xBG381x")
+		(lib_id "ECP5_BGA381_FT2232HQ_FIFO:LFE5U-25F-xBG381x")
 		(at 92.71 107.95 0)
 		(unit 1)
@@
 			)
 		)
-		(property "Footprint" "ECP5_TX_AUDIO:BGA-381_pitch0.8mm_dia0.4mm"
+		(property "Footprint" "ECP5_BGA381_FT2232HQ_FIFO:BGA-381_pitch0.8mm_dia0.4mm"
 			(at 88.9 -49.53 0)
 			(effects
